Commit message: Update for Isaac Sim and real Robot

File: config/so_100_arm.ros2_control.xacro (robot description, xacro)
@@ -11,6 +11,7 @@
                     <plugin>so_arm_100_controller/SOARM100Interface</plugin>
                     <param name="use_serial">true</param>
-                    <param name="serial_port">/dev/ttyUSB0</param>
+                    <param name="serial_port">/dev/ttyACM4</param>
                     <param name="serial_baudrate">1000000</param>
+                    <param name="calibration_file">/home/baxter/Documents/SO-100-arm/src/so_arm_100_hardware/config/calibration.yaml</param>
                 </xacro:unless>
             </hardware>

File: urdf/so_100_arm_5dof_hardware.urdf (robot description, URDF)
Before this commit: robot so_100_arm, 8 links, 7 joints
Joints:
- removed joint Gripper
- joint Elbow: limit (none) -> lower=-3.14 upper=-0.110 effort=100 velocity=1.0; type continuous -> revolute
- joint Shoulder_Pitch: limit (none) -> lower=-0.1 upper=3.14 effort=100 velocity=1.0; type continuous -> revolute
- joint Shoulder_Rotation: limit (none) -> lower=-3.14 upper=3.14 effort=100 velocity=1.0; origin xyz=0 -0.0452 0.0165 rpy=1.5708 0 -0.6 -> xyz=0 -0.0452 0.0165 rpy=-1.5708 0 00; type continuous -> revolute
- joint Wrist_Pitch: limit (none) -> lower=-3.14 upper=3.14 effort=100 velocity=1.0; type continuous -> revolute
- joint Wrist_Roll: limit (none) -> lower=0 upper=3.0 effort=100 velocity=1.0; type continuous -> revolute
